File: PCB/SF_01 Compute Board/SF_01 Compute Board.kicad_sch (KiCad schematic)
At the start: 30 parts, among them J1 SS-53200-001, J15 USB_C_Receptacle_USB2.0_16P, J2 Barrel_Jack, SW1 POWER, SW2 PI_BOOT, U1 CM4102008, U2 TPD4E02B04DQA, U3 TPD4E02B04DQA, U6 RT9742SNGV, U7 TPD4E02B04DQA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

Commit message: Changed Audio Multiplexer Circuit, Routed more
Parts:
- U8, U9: footprint Package_SON:Texas_X2SON-5_0.8x0.8mm_P0.48mm_RoutingVia -> Package_SON:Texas_X2SON-5_0.8x0.8mm_P0.48mm
Connections:
- net CM4_3.3V(OUTPUT) is gone; now on net 3V3: U1.78 (GPIO_VREF), U1.84 (CM4_3.3V(OUTPUT)), U1.86 (CM4_3.3V(OUTPUT))
- net +5V(INPUT): now also VR1.3 (INPUT); no longer C1.1, C2.1, D1.2 (A2), VR1.2 (OUTPUT_2), VR1.4 (OUTPUT_4)
- net GND: now also U1.SH1 (MOUNTING_PADS), U1.SH2 (MOUNTING_PADS), U1.SH3 (MOUNTING_PADS), U1.SH4 (MOUNTING_PADS)
- net HDMI_5V: now also C1.1, C2.1, D1.2 (A2)
- net VSYS: now also VR1.2 (OUTPUT_2), VR1.4 (OUTPUT_4); no longer VR1.3 (INPUT)
- net DATA2P: now reaches J1.1 (DATA2+), U1.170 (HDMI0_TX2_P), U3.1 (IO1), U3.10 (NC)
- net DATA2N: now reaches J1.3 (DATA2-), U1.172 (HDMI0_TX2_N), U3.2 (IO2), U3.9 (NC)
- net DATA1P: now reaches J1.4 (DATA1+), U1.176 (HDMI0_TX1_P), U3.4 (IO3), U3.7 (NC)
- net DATA1N: now reaches J1.6 (DATA1-), U1.178 (HDMI0_TX1_N), U3.5 (IO4), U3.6 (NC)
- net USBC1_DP: now reaches J15.A6 (D+), J15.B6 (D+), U1.105 (USB_P), U7.4 (IO3), U7.7 (NC)
- net USBC1_DN: now reaches J15.A7 (D-), J15.B7 (D-), U1.103 (USB_N), U7.5 (IO4), U7.6 (NC)
- net DATA0P: now reaches J1.7 (DATA0+), U1.182 (HDMI0_TX0_P), U2.1 (IO1), U2.10 (NC)
- net DATA0N: now reaches J1.9 (DATA0-), U1.184 (HDMI0_TX0_N), U2.2 (IO2), U2.9 (NC)
- net DATA3P: now reaches J1.10 (DATA3+), U1.188 (HDMI0_CLK_P), U2.4 (IO3), U2.7 (NC)
- net DATA3N: now reaches J1.12 (DATA3-), U1.190 (HDMI0_CLK_N), U2.5 (IO4), U2.6 (NC)

Commit message: Added USB Host control, Routed 1st amplifier
Parts:
- added C45, C47: 100nF, Capacitor_SMD:C_0603_1608Metric, symbol Device:C
- added C73: 22uF, Capacitor_SMD:CP_Elec_4x3, symbol Device:C_Polarized
- added R12: 10K, Resistor_SMD:R_0603_1608Metric, symbol Device:R
- added SW6: SW_DPDT_x2, Button_Switch_THT:SW_Push_2P2T_Toggle_CK_PVA2xxH1xxxxxxV2, symbol Switch:SW_DPDT_x2
- added U27: TPS2041B, Package_TO_SOT_SMD:SOT-23-5, symbol Power_Management:TPS2041B
Connections:
- net +5V(INPUT): now also C40.1, VR1.2 (OUTPUT_2), VR1.4 (OUTPUT_4), C45.2, R12.1, SW6.4 (A), U27.5 (IN); no longer C41.1, J15.A4 (VBUS), J15.A9 (VBUS), J15.B4 (VBUS), J15.B9 (VBUS), VR1.3 (INPUT)
- net 3V3: now also SW6.1 (A)
- net GND: now also C45.1, C47.1, C73.2, SW6.3 (C), SW6.6 (C), U27.2 (GND)
- net VSYS: now also C41.1, VR1.3 (INPUT); no longer C40.1, VR1.2 (OUTPUT_2), VR1.4 (OUTPUT_4)
- net at U1.101 (USB_OTG_ID): now also SW6.2 (B)
- new net: SW6.5 (B), U27.4 (~{EN})
- new net: R12.2, U27.3 (~{OC})
- new net VBUS: C47.2, C73.1, J15.A4 (VBUS), J15.A9 (VBUS), J15.B4 (VBUS), J15.B9 (VBUS), U27.1 (OUT)
Other:
- moved on the sheet: C3, C4, C5, J2, U6

Commit message: Finishing touches to PCB, add enclosure CAD files
Parts:
- SW6: footprint Button_Switch_THT:SW_Push_2P2T_Toggle_CK_PVA2xxH1xxxxxxV2 -> Button_Switch_SMD:SW_DPDT_CK_JS202011JCQN
Changed lines of the file:
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@@
 			)
 		)
-		(property "Footprint" "Button_Switch_THT:SW_Push_2P2T_Toggle_CK_PVA2xxH1xxxxxxV2"
+		(property "Footprint" "Button_Switch_SMD:SW_DPDT_CK_JS202011JCQN"
 			(at 278.13 146.05 0)
 			(hide yes)
@@
 			)
 		)
-		(property "Footprint" "Button_Switch_THT:SW_Push_2P2T_Toggle_CK_PVA2xxH1xxxxxxV2"
+		(property "Footprint" "Button_Switch_SMD:SW_DPDT_CK_JS202011JCQN"
 			(at 228.6 19.05 0)
 			(hide yes)
