File: PCB V1.1/SF_01 Compute Board/SF_01 Compute Board.kicad_pcb (KiCad board)
At the start: 4 copper layers, 128 x 128 mm, 329 parts, among them J1 SS-53200-001, J10 SUBWOOFER_6, J11 TWEETER_1, J12 TWEETER_2, J13 TWEETER_3, J14 TWEETER_4, J15 USB_C_Receptacle_USB2.0_16P, J2 Barrel_Jack, J3 UART, J5 SUBWOOFER_1, J6 SUBWOOFER_2, J7 SUBWOOFER_3, J8 SUBWOOFER_4, J9 SUBWOOFER_5, SW1 POWER, SW2 PI_BOOT, SW3 ESP_BOOT, SW4 ESP_RESET, SW6 SW_DPDT_x2, U1 CM4102008, U11 LP5907MFX-3.3, U12 TS5A3159AYZPR, U13 TS5A3159AYZPR, U14 PCM5102A, U15 TS5A3159AYZPR, U16 TS5A3159AYZPR, U17 TPA3116D2DAD, U18 TPA3116D2DAD, U19 TPA3116D2DAD, U2 TPD4E02B04DQA, U20 TPA3130D2DAPR, U21 TPA3130D2DAPR, U22 MPU-6050, U23 BME680, U24 TS5A3159AYZPR, U25 TS5A3159AYZPR, U26 TS5A3159AYZPR, U27 TPS2041B, U28 ESP32-WROVER-E-N16R8, U3 TPD4E02B04DQA, U5 PCM5102A, U6 RT9742SNGV, U7 TPD4E02B04DQA, U8 74LVC1G07, U9 74LVC1G07

Commit message: Fixed minor routing issues
Connections:
- R20 pad 2: WOOFER_MUTE -> TWEETER_MUTE
- R27 pad 2: WOOFER_MUTE -> TWEETER_MUTE
- R36 pad 2: WOOFER_MUTE -> TWEETER_MUTE
- U17 pad 12: WOOFER_MUTE -> TWEETER_MUTE
- U18 pad 12: WOOFER_MUTE -> TWEETER_MUTE
- U19 pad 12: WOOFER_MUTE -> TWEETER_MUTE
- U28 pad 12: WOOFER_MUTE -> TWEETER_MUTE
- U28 pad 8: TWEETER_MUTE -> ORIENTATION_SWITCH
Routing:
- net WOOFER_MUTE: track 208.0 -> 0.00 mm, vias 9 -> 0
- net TWEETER_MUTE: track 148.3 -> 346.3 mm, vias 3 -> 11
- net ORIENTATION_SWITCH: track 132.3 -> 145.5 mm
- net WFR_DIN: track 90.1 -> 92.1 mm
