File: PCB V1.1/SF_01 Compute Board/SF_01 Compute Board.kicad_pcb (KiCad board)
At the start: 4 copper layers, 128 x 128 mm, 345 parts, among them J1 SS-53200-001, J10 SUBWOOFER_6, J11 TWEETER_1, J12 TWEETER_2, J13 TWEETER_3, J14 TWEETER_4, J15 USB_C_Receptacle_USB2.0_16P, J2 Barrel_Jack, J3 UART, J5 SUBWOOFER_1, J6 SUBWOOFER_2, J7 SUBWOOFER_3, J8 SUBWOOFER_4, J9 SUBWOOFER_5, SW1 POWER, SW2 PI_BOOT, SW3 ESP_BOOT, SW4 ESP_RESET, SW6 SW_DPDT_x2, U1 CM4102008, U10 LP5907MFX-4.5, U11 LP5907MFX-3.3, U12 TS5A3159AYZPR, U13 TS5A3159AYZPR, U14 PCM5102A, U15 TS5A3159AYZPR, U16 TS5A3159AYZPR, U17 TPA3116D2DAD, U18 TPA3116D2DAD, U19 TPA3116D2DAD, U2 TPD4E02B04DQA, U20 TPA3130D2DAPR, U21 TPA3130D2DAPR, U22 MPU-6050, U23 BME680, U24 TS5A3159AYZPR, U25 TS5A3159AYZPR, U26 TS5A3159AYZPR, U27 TPS2041B, U28 ESP32-WROVER-E-N16R8, U3 TPD4E02B04DQA, U4 TPS54540DDAR, U5 PCM5102A, U6 RT9742SNGV, U7 TPD4E02B04DQA, U8 74LVC1G07, U9 74LVC1G07

Commit message: Fixed all PCB blocking issues, updated BOM
Parts:
- removed C127, C128, C140, C168: 1nF, Capacitor_SMD:C_0603_1608Metric
- added Q1: BSS138, Package_TO_SOT_SMD:SOT-23, F.Cu at (199.8, 44.7)
- added R7: 56K, Resistor_SMD:R_0603_1608Metric, F.Cu at (193.0, 44.1)
- C100, C101, C129, C191, C192: footprint Capacitor_SMD:C_0603_1608Metric -> Capacitor_SMD:C_1210_3225Metric
- D1: value SMAJ33CA -> SMAJ26A
- R17: value 100K -> 56K
- R25, R44, R49, R59: value 10K -> 100R
- U8, U9: footprint Package_SON:Texas_X2SON-5_0.8x0.8mm_P0.48mm -> Package_TO_SOT_SMD:SOT-23-5
- moved R17 36.2 mm to (193.0, 47.3)
- moved D1 24.7 mm to (175.0, 146.7), turned to 180 degrees
- moved U9 21.6 mm to (175.5, 131.4), turned to 90 degrees
- moved R6 16.4 mm to (179.1, 128.6), turned to 0 degrees
- moved D4 13.7 mm to (179.0, 126.7), turned to 180 degrees
- moved R3 12.7 mm to (193.0, 42.6)
- moved C191 11.8 mm to (151.8, 77.3), turned to 90 degrees
- moved C192 11.3 mm to (148.3, 77.3), turned to 90 degrees
- moved R65 11.1 mm to (193.0, 45.7)
- moved C129 4.64 mm to (151.1, 105.6), turned to -90 degrees
- moved C100 2.54 mm to (147.0, 103.7)
- moved U8 1.58 mm to (189.7, 145.3), turned to 0 degrees
- moved C3 1.20 mm to (182.0, 146.1)
- moved C101 0.81 mm to (147.0, 100.3)
- moved C78 0.50 mm to (116.9, 50.5)
Connections:
- D1 pad 1: GND -> VSYS
- D1 pad 2: HDMI_5V -> GND
- R17 pad 1: Net-(U17-FAULTZ) -> VBUS
- R17 pad 2: 3V3 -> Net-(J15-CC2)
- R3 pad 1: GND -> Net-(Q1-D)
- R65 pad 1: GND -> Net-(Q1-D)
- U20 pad 33: (no net) -> GND
- U21 pad 33: (no net) -> GND
Routing:
- net Net-(Q1-G): track 41.9 -> 115.4 mm, vias 2 -> 3
- net PWR_LED: track 47.1 -> 87.1 mm, vias 0 -> 2
- net 3V3: track 493.1 -> 469.4 mm, vias 31 -> 28
- net VBUS: track 103.4 -> 117.2 mm
- net Net-(J15-CC1): track 3.03 -> 16.2 mm
- net Net-(Q1-D): track 0.00 -> 12.0 mm
- net SYS_5V: track 457.7 -> 467.9 mm
- net VSYS: track 1080.5 -> 1089.5 mm, vias 282 -> 278
- net HDMI_5V: track 37.0 -> 28.3 mm, vias 4 -> 3
- net GND: track 1031.7 -> 1039.9 mm, vias 1360 -> 1348
- net Net-(U18-SYNC): track 23.2 -> 18.9 mm
- net Net-(U17-FAULTZ): track 10.7 -> 14.7 mm
- net Net-(U1A-RUN_PG): track 97.4 -> 93.5 mm
- net Net-(J15-CC2): track 12.5 -> 13.9 mm
- net Net-(U19-SYNC): track 6.32 -> 5.21 mm
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