File: PCB V1.1/SF_01 Compute Board/SF_01 Compute Board.kicad_pcb (KiCad board)
At the start: 4 copper layers, 128 x 128 mm, 343 parts, among them J1 SS-53200-001, J10 SUBWOOFER_6, J11 TWEETER_1, J12 TWEETER_2, J13 TWEETER_3, J14 TWEETER_4, J15 USB_C_Receptacle_USB2.0_16P, J2 Barrel_Jack, J3 UART, J5 SUBWOOFER_1, J6 SUBWOOFER_2, J7 SUBWOOFER_3, J8 SUBWOOFER_4, J9 SUBWOOFER_5, Q1 BSS138, SW1 POWER, SW2 PI_BOOT, SW3 ESP_BOOT, SW4 ESP_RESET, SW6 SW_DPDT_x2, U1 CM4102008, U10 LP5907MFX-4.5, U11 LP5907MFX-3.3, U12 TS5A3159AYZPR, U13 TS5A3159AYZPR, U14 PCM5102A, U15 TS5A3159AYZPR, U16 TS5A3159AYZPR, U17 TPA3116D2DAD, U18 TPA3116D2DAD, U19 TPA3116D2DAD, U2 TPD4E02B04DQA, U20 TPA3130D2DAPR, U21 TPA3130D2DAPR, U22 MPU-6050, U23 BME680, U24 TS5A3159AYZPR, U25 TS5A3159AYZPR, U26 TS5A3159AYZPR, U27 TPS2041B, U28 ESP32-WROVER-E-N16R8, U3 TPD4E02B04DQA, U4 TPS54540DDAR, U5 PCM5102A, U6 RT9742SNGV, U7 TPD4E02B04DQA, U8 74LVC1G07, U9 74LVC1G07

Commit message: Finished final version of PCB and BOM
Parts:
- removed U8: 74LVC1G07, Package_TO_SOT_SMD:SOT-23-5
- added C74: 100nF, Capacitor_SMD:C_0603_1608Metric, F.Cu at (191.1, 145.8)
- added R77: 10K, Resistor_SMD:R_0603_1608Metric, F.Cu at (188.5, 145.0)
- added R78: 220R, Resistor_SMD:R_0603_1608Metric, F.Cu at (155.0, 113.2)
- added TP1: TestPoint, TestPoint:TestPoint_Pad_3.0x3.0mm, F.Cu at (155.3, 116.1)
- added TP10: NEOPIXEL_DIN, TestPoint:TestPoint_Pad_D2.5mm, B.Cu at (151.9, 35.0)
- added TP11: WFR_BCK, TestPoint:TestPoint_Pad_3.0x3.0mm, B.Cu at (177.4, 68.3)
- added TP12: WFR_SCK, TestPoint:TestPoint_Pad_3.0x3.0mm, B.Cu at (182.5, 68.3)
- added TP13: TWT_DIN, TestPoint:TestPoint_Pad_3.0x3.0mm, B.Cu at (177.4, 73.4)
- added TP14: DRIVER_MUTE, TestPoint:TestPoint_Pad_D2.5mm, B.Cu at (169.1, 48.8)
- added TP15: WFR_DIN, TestPoint:TestPoint_Pad_3.0x3.0mm, B.Cu at (182.5, 73.4)
- added TP16: TestPoint, TestPoint:TestPoint_Pad_3.0x3.0mm, B.Cu at (182.5, 58.3)
- added TP17: TestPoint, TestPoint:TestPoint_Pad_D2.5mm, B.Cu at (182.8, 40.3)
- added TP18: TestPoint, TestPoint:TestPoint_Pad_3.0x3.0mm, B.Cu at (177.4, 58.3)
- added TP19: SDA, TestPoint:TestPoint_Pad_3.0x3.0mm, B.Cu at (177.4, 78.5)
- added TP2: TestPoint, TestPoint:TestPoint_Pad_3.0x3.0mm, F.Cu at (151.1, 116.1)
- added TP20: SCL, TestPoint:TestPoint_Pad_3.0x3.0mm, B.Cu at (182.5, 78.5)
- added TP21: TestPoint, TestPoint:TestPoint_Pad_D2.5mm, F.Cu at (87.0, 37.4)
- added TP23: TestPoint, TestPoint:TestPoint_Pad_D2.5mm, B.Cu at (81.8, 48.2)
- added TP24: TestPoint, TestPoint:TestPoint_Pad_D2.5mm, B.Cu at (189.7, 41.4)
- added TP25: TestPoint, TestPoint:TestPoint_Pad_D2.5mm, B.Cu at (186.2, 34.2)
- added TP3: TWT_L, TestPoint:TestPoint_Plated_Hole_D2.0mm, F.Cu at (88.7, 34.0)
- added TP4: TWT_R, TestPoint:TestPoint_Plated_Hole_D2.0mm, F.Cu at (85.0, 34.2)
- added TP5: WFR_L, TestPoint:TestPoint_Plated_Hole_D2.0mm, F.Cu at (87.4, 46.8)
- added TP6: WFR_R, TestPoint:TestPoint_Plated_Hole_D2.0mm, F.Cu at (91.1, 46.8)
- added TP7: ORIENTATION, TestPoint:TestPoint_Pad_D2.5mm, B.Cu at (177.5, 37.0)
- added TP8: TWT_BCK, TestPoint:TestPoint_Pad_3.0x3.0mm, B.Cu at (177.4, 63.3)
- added TP9: TWT_LRCK, TestPoint:TestPoint_Pad_3.0x3.0mm, B.Cu at (182.5, 63.3)
- C100, C101, C129: value 10uF/25V -> 10uF/50V
- moved C123 3.24 mm to (90.2, 132.7), turned to 90 degrees
- moved C84 1.10 mm to (106.4, 65.9), turned to 180 degrees
Connections:
- SW1 pad 1: Net-(SW1-Pad1) -> Net-(U1A-GPIO3)
- SW1 pad 2: Net-(U1A-GLOBAL_EN) -> GND
- U1 pad 56: unconnected-(U1A-GPIO3-Pad56) -> Net-(U1A-GPIO3)
Routing:
- net Net-(U1A-GPIO3): track 0.00 -> 102.2 mm, vias 0 -> 2
- net SYS_5V: track 467.9 -> 417.8 mm, vias 59 -> 57
- net WFR_DIN: track 92.3 -> 135.8 mm, vias 2 -> 3
- net TWT_DIN: track 64.4 -> 103.6 mm, vias 0 -> 1
- net WFR_SCK: track 67.4 -> 106.2 mm
- net TWT_LRCK: track 76.8 -> 114.9 mm
- net Net-(C10-Pad1): track 3.31 -> 37.1 mm, vias 0 -> 1
- net 3V3: track 469.4 -> 502.0 mm, vias 28 -> 30
- net WFR_BCK: track 67.7 -> 99.4 mm
- net SCL: track 128.2 -> 155.4 mm
- net Net-(U4-SW): track 14.8 -> 37.6 mm, vias 0 -> 12
- net SDA: track 127.8 -> 150.2 mm
- net WFR_LRCK: track 85.0 -> 102.3 mm
- net GND: track 1039.9 -> 1052.9 mm, vias 1348 -> 1334
- net Net-(C188-Pad1): track 4.57 -> 16.5 mm
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Other:
- board text added: "3V3"
- board text added: "DAC enable"
- board text added: "Driver mute"
- board text added: "GND"
- board text added: "NeoPixel Din"
- board text added: "Orientation"
- board text added: "Pi RUN_PG"
- board text added: "Pi USB Switch -->"
- board text added: "Pi global enable"
- board text added: "SCL"
- board text added: "SDA"
- board text added: "SF_01 Mainboard v1.5"
- board text added: "Tweeter Bclock"
- board text added: "Tweeter Din"
- board text added: "Tweeter LRclock"
- board text added: "Tweeter Sclock"
- board text added: "Woofer Bclock"
- board text added: "Woofer Din"
- board text added: "Woofer LRclock"
- board text added: "Woofer Sclock"
- board text removed: "Raspberry Pi USB Switch"
- board text removed: "SF_01 Mainboard"
- board text removed: "Triangulate"
- board text removed: "Version 1.5"
