File: PCB V1.1/SF_01 Compute Board/audioCircuit.kicad_sch (KiCad schematic)
At the start: 130 parts, among them J10 SUBWOOFER_6, J5 SUBWOOFER_1, J6 SUBWOOFER_2, J7 SUBWOOFER_3, J8 SUBWOOFER_4, J9 SUBWOOFER_5, U17 TPA3116D2DAD, U18 TPA3116D2DAD, U19 TPA3116D2DAD

Commit message: Fixed major issues with power rails
Parts:
- removed R17: 100K, Resistor_SMD:R_0603_1608Metric, symbol Device:R
- added R50: 100K, Resistor_SMD:R_0603_1608Metric, symbol Device:R
- C104, C110, C51, C54, C78, C83: footprint Capacitor_SMD:CP_Elec_5x5.3 -> Capacitor_SMD:CP_Elec_6.3x9.9
Connections:
- net at R30.1: now also U18.12 (MUTE); no longer U18.3 (FAULTZ)
- net at R39.1: now also U17.12 (MUTE); no longer U19.3 (FAULTZ)
- net at U17.3 (FAULTZ): now also R16.2, U17.2 (SDZ)
- removed net 3V3: R16.2, R26.2, R30.2, R35.2, R39.2, U17.2 (SDZ), U18.2 (SDZ), U19.2 (SDZ)
- net WOOFER_MUTE renamed DRIVER_MUTE
- net DRIVER_MUTE: now also R30.2, R39.2, R50.2; no longer U17.12 (MUTE), U18.12 (MUTE), U19.12 (MUTE)
- new net: R26.2, U18.2 (SDZ), U18.3 (FAULTZ)
- new net: R50.1, U19.12 (MUTE)
- new net: R35.2, U19.2 (SDZ), U19.3 (FAULTZ)
Other:
- moved on the sheet: R20, R36

Commit message: Fixed all PCB blocking issues, updated BOM
Parts:
- removed C127, C128: 1nF, Capacitor_SMD:C_0603_1608Metric, symbol Device:C
- R25, R44: value 10K -> 100R
