File: PCB V1.1/SF_01 Compute Board/tweeterAmps.kicad_sch (KiCad schematic)
At the start: 86 parts, among them J11 TWEETER_1, J12 TWEETER_2, J13 TWEETER_3, J14 TWEETER_4, U20 TPA3130D2DAPR, U21 TPA3130D2DAPR

Commit message: Fixed major issues with power rails
Parts:
- removed R50: 100K, Resistor_SMD:R_0603_1608Metric, symbol Device:R
- added R76: 100K, Resistor_SMD:R_0603_1608Metric, symbol Device:R
- C133, C139, C161, C167: footprint Capacitor_SMD:CP_Elec_5x5.3 -> Capacitor_SMD:CP_Elec_6.3x9.9
Connections:
- net at R60.1: now also U20.12 (MUTE); no longer U21.3 (FAULTZ)
- net at U20.3 (FAULTZ): now also R45.2, U20.2 (SDZ)
- removed net 3V3: R45.2, R55.2, R60.2, U20.2 (SDZ), U21.2 (SDZ)
- net TWEETER_MUTE renamed DRIVER_MUTE
- net DRIVER_MUTE: now also R60.2, R76.2; no longer U20.12 (MUTE), U21.12 (MUTE)
- new net: R76.1, U21.12 (MUTE)
- new net: R55.2, U21.2 (SDZ), U21.3 (FAULTZ)
Other:
- moved on the sheet: R46, R56

Commit message: Fixed all PCB blocking issues, updated BOM
Parts:
- removed C140, C168: 1nF, Capacitor_SMD:C_0603_1608Metric, symbol Device:C
- R49, R59: value 10K -> 100R
