File: PCB V1.1/SF_01 Compute Board/ESP32Wrover.kicad_sch (KiCad schematic)
At the start: 9 parts, among them J3 UART, SW3 ESP_BOOT, SW4 ESP_RESET, U28 ESP32-WROVER-E-N16R8

Commit message: Fixed minor routing issues
Connections:
- net WOOFER_MUTE is gone; now on net TWEETER_MUTE: U28.12 (IO27)
- net TWEETER_MUTE: no longer U28.8 (IO32)
- new net ORIENTATION_SWITCH: U28.8 (IO32)
Changed lines of the file:
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@@
 	(wire
 		(pts
-			(xy 60.96 83.82) (xy 74.93 83.82)
+			(xy 43.18 83.82) (xy 74.93 83.82)
 		)
 		(stroke
@@
 	(wire
 		(pts
+			(xy 38.1 91.44) (xy 38.1 93.98)
+		)
+		(stroke
+			(width 0)
+			(type default)
+		)
+	)
+	(wire
+		(pts
 			(xy 36.83 43.18) (xy 36.83 26.67)
 		)
@@
 	(wire
 		(pts
-			(xy 59.69 93.98) (xy 74.93 93.98)
+			(xy 38.1 93.98) (xy 74.93 93.98)
 		)
 		(stroke
@@
 	(global_label "TWEETER_MUTE"
 		(shape input)
-		(at 60.96 83.82 180)
-		(fields_autoplaced yes)
-		(effects
-			(font
-				(size 1.27 1.27)
-			)
-			(justify right)
-		)
-		(property "Intersheetrefs" "${INTERSHEET_REFS}"
-			(at 44.0051 83.82 0)
+		(at 38.1 91.44 180)
+		(fields_autoplaced yes)
+		(effects
+			(font
+				(size 1.27 1.27)
+			)
+			(justify right)
+		)
+		(property "Intersheetrefs" "${INTERSHEET_REFS}"
+			(at 21.1451 91.44 0)
 			(hide yes)
 			(show_name no)
@@
 	(global_label "WOOFER_MUTE"
 		(shape input)
-		(at 59.69 93.98 180)
-		(fields_autoplaced yes)
-		(effects
-			(font
-				(size 1.27 1.27)
-			)
-			(justify right)
-		)
-		(property "Intersheetrefs" "${INTERSHEET_REFS}"
-			(at 43.2187 93.98 0)
+		(at 38.1 93.98 180)
+		(fields_autoplaced yes)
+		(effects
+			(font
+				(size 1.27 1.27)
+			)
+			(justify right)
+		)
+		(property "Intersheetrefs" "${INTERSHEET_REFS}"
+			(at 21.6287 93.98 0)
 			(hide yes)
 			(show_name no)
@@
 			)
 		)
+	)
+	(global_label "ORIENTATION_SWITCH"
+		(shape input)
+		(at 43.18 83.82 180)
+		(fields_autoplaced yes)
+		(effects
+			(font
+				(size 1.27 1.27)
+			)
+			(justify right)
+		)
+		(property "Intersheetrefs" "${INTERSHEET_REFS}"
+			(at 20.419 83.82 0)
+			(hide yes)
+			(show_name no)
+			(do_not_autoplace no)
+			(effects
+				(font
+					(size 1.27 1.27)
+				)
+				(justify right)
+			)
+		)

Commit message: Fixed major issues with power rails
Connections:
- net TWEETER_MUTE renamed DRIVER_MUTE
Changed lines of the file:
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@@
 	(wire
 		(pts
-			(xy 60.96 86.36) (xy 74.93 86.36)
+			(xy 59.69 86.36) (xy 74.93 86.36)
 		)
 		(stroke
@@
 	(wire
 		(pts
-			(xy 43.18 83.82) (xy 74.93 83.82)
+			(xy 59.69 83.82) (xy 74.93 83.82)
 		)
 		(stroke
@@
 	(wire
 		(pts
-			(xy 38.1 91.44) (xy 38.1 93.98)
-		)
-		(stroke
-			(width 0)
-			(type default)
-		)
-	)
-	(wire
-		(pts
 			(xy 36.83 43.18) (xy 36.83 26.67)
 		)
@@
 	(wire
 		(pts
-			(xy 57.15 96.52) (xy 74.93 96.52)
+			(xy 59.69 96.52) (xy 74.93 96.52)
 		)
 		(stroke
@@
 	(wire
 		(pts
-			(xy 38.1 93.98) (xy 74.93 93.98)
+			(xy 59.69 93.98) (xy 74.93 93.98)
 		)
 		(stroke
@@
 	(wire
 		(pts
-			(xy 120.65 119.38) (xy 138.43 119.38)
+			(xy 120.65 119.38) (xy 129.54 119.38)
 		)
 		(stroke
@@
 	(global_label "TWT_DIN"
 		(shape input)
-		(at 57.15 96.52 180)
+		(at 59.69 96.52 180)
 		(fields_autoplaced yes)
 		(effects
@@
 		)
 		(property "Intersheetrefs" "${INTERSHEET_REFS}"
-			(at 46.6053 96.52 0)
+			(at 49.1453 96.52 0)
 			(hide yes)
 			(show_name no)
@@
 	(global_label "NEOPIXEL_DIN"
 		(shape input)
-		(at 60.96 86.36 180)
+		(at 59.69 86.36 180)
 		(fields_autoplaced yes)
 		(effects
@@
 		)
 		(property "Intersheetrefs" "${INTERSHEET_REFS}"
-			(at 44.7305 86.36 0)
+			(at 43.4605 86.36 0)
 			(hide yes)
 			(show_name no)
@@
 	(global_label "DAC_EN"
 		(shape input)
-		(at 138.43 119.38 0)
+		(at 129.54 119.38 0)
 		(fields_autoplaced yes)
 		(effects
@@
 		)
 		(property "Intersheetrefs" "${INTERSHEET_REFS}"
-			(at 148.4909 119.38 0)
+			(at 139.6009 119.38 0)
 			(hide yes)
 			(show_name no)
@@
 		)
 	)
-	(global_label "TWEETER_MUTE"
-		(shape input)
-		(at 38.1 91.44 180)
+	(global_label "DRIVER_MUTE"
+		(shape input)
+		(at 59.69 93.98 180)
 		(fields_autoplaced yes)
 		(effects
@@
 		)
 		(property "Intersheetrefs" "${INTERSHEET_REFS}"
-			(at 21.1451 91.44 0)
+			(at 44.1863 93.98 0)
 			(hide yes)
 			(show_name no)
@@
 		)
 	)
-	(global_label "WOOFER_MUTE"
-		(shape input)
-		(at 38.1 93.98 180)
+	(global_label "SDA"
+		(shape input)
+		(at 128.27 101.6 0)
+		(fields_autoplaced yes)
+		(effects
+			(font
+				(size 1.27 1.27)
+			)
+			(justify left)
+		)
+		(property "Intersheetrefs" "${INTERSHEET_REFS}"
+			(at 134.8233 101.6 0)
+			(hide yes)
+			(show_name no)
+			(do_not_autoplace no)
+			(effects
+				(font
+					(size 1.27 1.27)
+				)
+				(justify left)
+			)
+		)
+	)
+	(global_label "ORIENTATION_SWITCH"
+		(shape input)
+		(at 59.69 83.82 180)
 		(fields_autoplaced yes)
 		(effects
@@
 		)
 		(property "Intersheetrefs" "${INTERSHEET_REFS}"
-			(at 21.6287 93.98 0)
-			(hide yes)
-			(show_name no)
-			(do_not_autoplace no)
-			(effects
-				(font
-					(size 1.27 1.27)
-				)
-				(justify right)
-			)
-		)
-	)
-	(global_label "SDA"
-		(shape input)
-		(at 128.27 101.6 0)
-		(fields_autoplaced yes)
-		(effects
-			(font
-				(size 1.27 1.27)
-			)
-			(justify left)
-		)
-		(property "Intersheetrefs" "${INTERSHEET_REFS}"
-			(at 134.8233 101.6 0)
-			(hide yes)
-			(show_name no)
-			(do_not_autoplace no)
-			(effects
-				(font
-					(size 1.27 1.27)
-				)
-				(justify left)
-			)
-		)
-	)
-	(global_label "ORIENTATION_SWITCH"
-		(shape input)
-		(at 43.18 83.82 180)
-		(fields_autoplaced yes)
-		(effects
-			(font
-				(size 1.27 1.27)
-			)
-			(justify right)
-		)
-		(property "Intersheetrefs" "${INTERSHEET_REFS}"
-			(at 20.419 83.82 0)
-			(hide yes)
-			(show_name no)
+			(at 36.929 83.82 0)
+			(hide yes)
+			(show_name no)

Commit message: Finished final version of PCB and BOM
Parts:
- added TP10: NEOPIXEL_DIN, TestPoint:TestPoint_Pad_D2.5mm, symbol Connector:TestPoint
- added TP11: WFR_BCK, TestPoint:TestPoint_Pad_3.0x3.0mm, symbol Connector:TestPoint
- added TP12: WFR_SCK, TestPoint:TestPoint_Pad_3.0x3.0mm, symbol Connector:TestPoint
- added TP13: TWT_DIN, TestPoint:TestPoint_Pad_3.0x3.0mm, symbol Connector:TestPoint
- added TP14: DRIVER_MUTE, TestPoint:TestPoint_Pad_D2.5mm, symbol Connector:TestPoint
- added TP15: WFR_DIN, TestPoint:TestPoint_Pad_3.0x3.0mm, symbol Connector:TestPoint
- added TP16, TP17, TP18: TestPoint, TestPoint:TestPoint_Pad_D2.5mm, symbol Connector:TestPoint
- added TP19: SDA, TestPoint:TestPoint_Pad_3.0x3.0mm, symbol Connector:TestPoint
- added TP20: SCL, TestPoint:TestPoint_Pad_3.0x3.0mm, symbol Connector:TestPoint
- added TP8: TWT_BCK, TestPoint:TestPoint_Pad_3.0x3.0mm, symbol Connector:TestPoint
- added TP9: TWT_LRCK, TestPoint:TestPoint_Pad_3.0x3.0mm, symbol Connector:TestPoint
Connections:
- net DAC_EN: now also TP17.1
- net DRIVER_MUTE: now also TP14.1
- net NEOPIXEL_DIN: now also TP10.1
- net SCL: now also TP20.1
- net SDA: now also TP19.1
- net TWT_BCK: now also TP8.1
- net TWT_DIN: now also TP13.1
- net TWT_LRCK: now also TP9.1
- net TWT_SCK: now also TP16.1
- net WFR_BCK: now also TP11.1
- net WFR_DIN: now also TP15.1
- net WFR_LRCK: now also TP18.1
- net WFR_SCK: now also TP12.1
