File: PCB V1.1/SF_01 Compute Board/SF_01 Compute Board.kicad_sch (KiCad schematic)
At the start: 36 parts, among them J1 SS-53200-001, J15 USB_C_Receptacle_USB2.0_16P, J2 Barrel_Jack, SW1 POWER, SW2 PI_BOOT, SW6 SW_DPDT_x2, U1 CM4102008, U2 TPD4E02B04DQA, U27 TPS2041B, U3 TPD4E02B04DQA, U6 RT9742SNGV, U7 TPD4E02B04DQA, U8 74LVC1G07, U9 74LVC1G07

Commit message: Fixed major issues with power rails
Parts:
- removed C3, C40: 10uF, Capacitor_SMD:CP_Elec_4x3, symbol Device:C_Polarized
- removed C4, C45, C47, C5: 100nF, Capacitor_SMD:C_0603_1608Metric, symbol Device:C
- removed C41: 10uF (Tantalum), Capacitor_Tantalum_SMD:CP_EIA-1608-08_AVX-J, symbol Device:C_Polarized
- removed C73: 22uF, Capacitor_SMD:CP_Elec_4x3, symbol Device:C_Polarized
- removed J2: Barrel_Jack, Connector_BarrelJack:BarrelJack_SwitchcraftConxall_RAPC10U_Horizontal, symbol Connector:Barrel_Jack
- removed R12: 10K, Resistor_SMD:R_0603_1608Metric, symbol Device:R
- removed unit 2 of SW6
- removed U27: TPS2041B, Package_TO_SOT_SMD:SOT-23-5, symbol Power_Management:TPS2041B
- removed U6: RT9742SNGV, Package_TO_SOT_SMD:SOT-23-3, symbol Power_Management:RT9742SNGV
- removed VR1: LM1085ISX-5.0_NOPB, LM1085ISX-5.0_NOPB:TO254P1435X464-4N, symbol LM1085ISX-5.0/NOPB:LM1085ISX-5.0_NOPB
Other:
- added sheet Power Rails (powerRails.kicad_sch)

Commit message: Fixed all PCB blocking issues, updated BOM
Parts:
- removed D1: SMAJ33CA, Diode_SMD:D_SMA, symbol Diode:SMAJ33CA
- added Q1: BSS138, Package_TO_SOT_SMD:SOT-23, symbol Transistor_FET:BSS138
- added R17, R7: 56K, Resistor_SMD:R_0603_1608Metric, symbol Device:R
- U8, U9: footprint Package_SON:Texas_X2SON-5_0.8x0.8mm_P0.48mm -> Package_TO_SOT_SMD:SOT-23-5
Connections:
- net GND: now also Q1.2 (S); no longer R3.1, R65.1
- net VBUS: now also R17.1, R7.1
- net at J15.B5 (CC2), R65.2: now also R17.2
- net at J15.A5 (CC1), R3.2: now also R7.2
- net at SW6.2 (B), U1.101 (USB_OTG_ID): now also Q1.1 (G)
- new net: Q1.3 (D), R3.1, R65.1
Other:
- moved on the sheet: R1, R2, R3, R65

Commit message: Finished final version of PCB and BOM
Parts:
- removed U8: 74LVC1G07, Package_TO_SOT_SMD:SOT-23-5, symbol 74xGxx:74LVC1G07
- added C74: 100nF, Capacitor_SMD:C_0603_1608Metric, symbol Device:C
- added R77: 10K, Resistor_SMD:R_0603_1608Metric, symbol Device:R
- added R78: 220R, Resistor_SMD:R_0603_1608Metric, symbol Device:R
- added TP1, TP2: TestPoint, TestPoint:TestPoint_Pad_3.0x3.0mm, symbol Connector:TestPoint
Connections:
- net 3V3: now also R77.1
- net GND: now also SW1.2, C74.2
- net at SW1.1: now also U1.56 (GPIO3), C74.1, R77.2
- net at U1.99 (GLOBAL_EN): now also TP2.1; no longer SW1.2
- net at U1.92 (RUN_PG): now also R78.1
- new net: R78.2, TP1.1
