File: PCB V1.1/SF_01 Compute Board/esp32Circuit.kicad_sch (KiCad schematic)
At the start: 55 parts, among them U11 LP5907MFX-3.3, U12 TS5A3159AYZPR, U13 TS5A3159AYZPR, U14 PCM5102A, U15 TS5A3159AYZPR, U16 TS5A3159AYZPR, U24 TS5A3159AYZPR, U25 TS5A3159AYZPR, U26 TS5A3159AYZPR, U5 PCM5102A

Commit message: Fixed major issues with power rails
Parts:
- removed C12, C13: 1uF, Capacitor_SMD:C_0603_1608Metric, symbol Device:C
- removed U11: LP5907MFX-3.3, Package_TO_SOT_SMD:SOT-23-5, symbol Regulator_Linear:LP5907MFX-3.3
Connections:
- net 3V3_A: no longer U12.B2 (V+), U13.B2 (V+), U15.B2 (V+), U16.B2 (V+), U24.B2 (V+), U25.B2 (V+), U26.B2 (V+)
- new net 4V5_A: U12.B2 (V+), U13.B2 (V+), U15.B2 (V+), U16.B2 (V+), U24.B2 (V+), U25.B2 (V+), U26.B2 (V+)

Commit message: Finished final version of PCB and BOM
Parts:
- added TP21, TP22, TP23, TP24, TP25, TP26: TestPoint, TestPoint:TestPoint_Pad_D2.5mm, symbol Connector:TestPoint
- added TP3: TWT_L, TestPoint:TestPoint_Plated_Hole_D2.0mm, symbol Connector:TestPoint
- added TP4: TWT_R, TestPoint:TestPoint_Plated_Hole_D2.0mm, symbol Connector:TestPoint
- added TP5: WFR_L, TestPoint:TestPoint_Plated_Hole_D2.0mm, symbol Connector:TestPoint
- added TP6: WFR_R, TestPoint:TestPoint_Plated_Hole_D2.0mm, symbol Connector:TestPoint
- added TP7: ORIENTATION, TestPoint:TestPoint_Pad_D2.5mm, symbol Connector:TestPoint
Connections:
- net 3V3: now also TP25.1
- net GND: now also TP21.1, TP22.1, TP23.1, TP24.1, TP26.1
- net ORIENTATION_SWITCH: now also TP7.1
- net at C188.1, C35.2, R10.2: now also TP5.1
- net at C190.1, C36.1, R11.2: now also TP6.1
- net at C11.2, C158.1, R8.2: now also TP3.1
- net at C10.1, C157.1, R9.2: now also TP4.1
Other:
- note removed: "This too complicated to explain"
- moved on the sheet: C158
